File: hardware/KiCAD/pc080/pc080.kicad_pcb (KiCad board)
At the start: 2 copper layers, 46 x 9.2 mm, 5 parts, among them J1 Conn_02x10_Top_Bottom, J4 Conn_01x05, J5 Conn_01x05, J6 Conn_01x05, J7 Conn_01x05

Commit message: Generated artwork. Tidied BoM. Got quote from PCBtrain
Parts:
- J6: moved to F.Cu
- moved J7 23.1 mm to (156.5, 70.9), turned to -90 degrees
- moved J6 21.5 mm to (149.0, 70.9), turned to -90 degrees
- moved J4 14.2 mm to (141.3, 70.9)
- moved J5 8.81 mm to (133.3, 70.9)
Connections:
- J1 pad 10: unconnected-(J1-Pin_10-Pad10) -> Net-(J1-Pin_10)
- J1 pad 12: unconnected-(J1-Pin_12-Pad12) -> Net-(J1-Pin_12)
- J1 pad 13: unconnected-(J1-Pin_13-Pad13) -> Net-(J1-Pin_13)
- J1 pad 14: unconnected-(J1-Pin_14-Pad14) -> Net-(J1-Pin_14)
- J1 pad 16: unconnected-(J1-Pin_16-Pad16) -> Net-(J1-Pin_16)
- J1 pad 17: unconnected-(J1-Pin_17-Pad17) -> Net-(J1-Pin_17)
- J1 pad 18: unconnected-(J1-Pin_18-Pad18) -> Net-(J1-Pin_18)
- J1 pad 19: unconnected-(J1-Pin_19-Pad19) -> Net-(J1-Pin_19)
- J1 pad 20: unconnected-(J1-Pin_20-Pad20) -> Net-(J1-Pin_20)
- J1 pad 4: unconnected-(J1-Pin_4-Pad4) -> Net-(J1-Pin_4)
- J1 pad 5: unconnected-(J1-Pin_5-Pad5) -> Net-(J1-Pin_5)
- J1 pad 6: unconnected-(J1-Pin_6-Pad6) -> Net-(J1-Pin_6)
- J1 pad 7: unconnected-(J1-Pin_7-Pad7) -> Net-(J1-Pin_7)
- J1 pad 8: unconnected-(J1-Pin_8-Pad8) -> Net-(J1-Pin_8)
- J1 pad 9: unconnected-(J1-Pin_9-Pad9) -> Net-(J1-Pin_9)
- J4 pad 4: unconnected-(J4-Pin_4-Pad4) -> Net-(J1-Pin_4)
- J4 pad 5: unconnected-(J4-Pin_5-Pad5) -> Net-(J1-Pin_5)
- J5 pad 1: unconnected-(J5-Pin_1-Pad1) -> Net-(J1-Pin_6)
- J5 pad 2: unconnected-(J5-Pin_2-Pad2) -> Net-(J1-Pin_7)
- J5 pad 3: unconnected-(J5-Pin_3-Pad3) -> Net-(J1-Pin_8)
- J5 pad 4: unconnected-(J5-Pin_4-Pad4) -> Net-(J1-Pin_9)
- J5 pad 5: unconnected-(J5-Pin_5-Pad5) -> Net-(J1-Pin_10)
- J6 pad 1: Net-(J1-Pin_11) -> Net-(J1-Pin_15)
- J6 pad 2: unconnected-(J6-Pin_2-Pad2) -> Net-(J1-Pin_14)
- J6 pad 3: unconnected-(J6-Pin_3-Pad3) -> Net-(J1-Pin_13)
- J6 pad 4: unconnected-(J6-Pin_4-Pad4) -> Net-(J1-Pin_12)
- J6 pad 5: Net-(J1-Pin_15) -> Net-(J1-Pin_11)
- J7 pad 1: unconnected-(J7-Pin_1-Pad1) -> Net-(J1-Pin_20)
- J7 pad 2: unconnected-(J7-Pin_2-Pad2) -> Net-(J1-Pin_19)
- J7 pad 3: unconnected-(J7-Pin_3-Pad3) -> Net-(J1-Pin_18)
- J7 pad 4: unconnected-(J7-Pin_4-Pad4) -> Net-(J1-Pin_17)
- J7 pad 5: unconnected-(J7-Pin_5-Pad5) -> Net-(J1-Pin_16)
Routing:
- net Net-(J1-Pin_10): track 0.00 -> 30.8 mm, vias 0 -> 1
- net Net-(J1-Pin_9): track 0.00 -> 30.3 mm, vias 0 -> 1
- net Net-(J1-Pin_8): track 0.00 -> 30.1 mm, vias 0 -> 1
- net Net-(J1-Pin_7): track 0.00 -> 30.0 mm, vias 0 -> 1
- net Net-(J1-Pin_6): track 0.00 -> 30.0 mm, vias 0 -> 1
- net Net-(J1-Pin_3): track 0.00 -> 22.8 mm, vias 0 -> 1
- net Net-(J1-Pin_2): track 0.00 -> 22.6 mm, vias 0 -> 1
- net Net-(J1-Pin_1): track 0.00 -> 22.6 mm, vias 0 -> 1
- net Net-(J1-Pin_4): track 0.00 -> 22.3 mm, vias 0 -> 1
- net Net-(J1-Pin_5): track 0.00 -> 21.7 mm, vias 0 -> 1
- net Net-(J1-Pin_15): track 0.00 -> 17.0 mm
- net Net-(J1-Pin_14): track 0.00 -> 16.7 mm
- net Net-(J1-Pin_13): track 0.00 -> 16.0 mm
- net Net-(J1-Pin_12): track 0.00 -> 15.8 mm
- net Net-(J1-Pin_11): track 0.00 -> 15.6 mm
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Other:
- board size 46 x 9.2 mm -> 45.9 x 11.9 mm
- board text added: "Based on TE Direct attach cable 14280017"
- board text added: "Use with 0.3mm thick FFC . e.g. Molex 98266-0105"
- board text added: "pc080_sfp_plug DUNE Sept 26"
