File: hardware/KiCAD/pc080/pc080.kicad_sch (KiCad schematic)
At the start: 5 parts, among them J1 Conn_02x10_Top_Bottom, J4 Conn_01x05, J5 Conn_01x05, J6 Conn_01x05, J7 Conn_01x05

Commit message: Generated artwork. Tidied BoM. Got quote from PCBtrain
Connections:
- net at J4.4 (Pin_4): now also J1.4 (Pin_4)
- net at J4.5 (Pin_5): now also J1.5 (Pin_5)
- net at J5.1 (Pin_1): now also J1.6 (Pin_6)
- net at J5.2 (Pin_2): now also J1.7 (Pin_7)
- net at J5.3 (Pin_3): now also J1.8 (Pin_8)
- net at J5.4 (Pin_4): now also J1.9 (Pin_9)
- net at J5.5 (Pin_5): now also J1.10 (Pin_10)
- net at J1.11 (Pin_11): now also J6.5 (Pin_5); no longer J6.1 (Pin_1)
- net at J1.12 (Pin_12): now also J6.4 (Pin_4)
- net at J1.13 (Pin_13): now also J6.3 (Pin_3)
- net at J1.14 (Pin_14): now also J6.2 (Pin_2)
- net at J1.15 (Pin_15): now also J6.1 (Pin_1); no longer J6.5 (Pin_5)
- net at J1.16 (Pin_16): now also J7.5 (Pin_5)
- net at J1.17 (Pin_17): now also J7.4 (Pin_4)
- net at J1.18 (Pin_18): now also J7.3 (Pin_3)
- net at J1.19 (Pin_19): now also J7.2 (Pin_2)
- net at J1.20 (Pin_20): now also J7.1 (Pin_1)
Other:
- note added: "5 way FFC connectors"
- note added: "SFP plug (PCB edge connector)"
- company: (none) -> University of Bristol
- title: (none) -> SFP Plug breakout
Changed lines of the file:
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@@
 	(generator_version "10.0")
 	(paper "A4")
+	(title_block
+		(title "SFP Plug breakout")
+		(date "2026-09-28")
+		(rev "1")
+		(company "University of Bristol")
+		(comment 1 "David.Cussans@bristol.ac.uk")
+	)
+	(text "SFP plug\n(PCB edge connector)"
+		(exclude_from_sim no)
+		(at 143.256 91.44 0)
+		(effects
+			(font
+				(size 1.27 1.27)
+			)
+		)
+	)
+	(text "5 way FFC\nconnectors"
+		(exclude_from_sim no)
+		(at 114.3 91.694 0)
+		(effects
+			(font
+				(size 1.27 1.27)
+			)
+		)
+	)
+	(wire
+		(pts
+			(xy 148.59 85.09) (xy 160.02 85.09)
+		)
+		(stroke
+			(width 0)
+			(type default)
+		)
+	)
 	(wire
 		(pts
@@
 	(wire
 		(pts
+			(xy 119.38 69.85) (xy 135.89 69.85)
+		)
+		(stroke
+			(width 0)
+			(type default)
+		)
+	)
+	(wire
+		(pts
+			(xy 119.38 82.55) (xy 135.89 82.55)
+		)
+		(stroke
+			(width 0)
+			(type default)
+		)
+	)
+	(wire
+		(pts
+			(xy 119.38 77.47) (xy 135.89 77.47)
+		)
+		(stroke
+			(width 0)
+			(type default)
+		)
+	)
+	(wire
+		(pts
 			(xy 119.38 64.77) (xy 135.89 64.77)
 		)
@@
 	(wire
 		(pts
+			(xy 148.59 74.93) (xy 160.02 74.93)
+		)
+		(stroke
+			(width 0)
+			(type default)
+		)
+	)
+	(wire
+		(pts
+			(xy 148.59 67.31) (xy 160.02 67.31)
+		)
+		(stroke
+			(width 0)
+			(type default)
+		)
+	)
+	(wire
+		(pts
+			(xy 119.38 74.93) (xy 135.89 74.93)
+		)
+		(stroke
+			(width 0)
+			(type default)
+		)
+	)
+	(wire
+		(pts
 			(xy 119.38 67.31) (xy 135.89 67.31)
 		)
@@
 	(wire
 		(pts
+			(xy 148.59 64.77) (xy 160.02 64.77)
+		)
+		(stroke
+			(width 0)
+			(type default)
+		)
+	)
+	(wire
+		(pts
 			(xy 148.59 62.23) (xy 160.02 62.23)
+		)
+		(stroke
+			(width 0)
+			(type default)
+		)
+	)
+	(wire
+		(pts
+			(xy 148.59 82.55) (xy 160.02 82.55)
+		)
+		(stroke
+			(width 0)
+			(type default)
+		)
+	)
+	(wire
+		(pts
+			(xy 119.38 85.09) (xy 135.89 85.09)
+		)
+		(stroke
+			(width 0)
+			(type default)
+		)
+	)
+	(wire
+		(pts
+			(xy 119.38 80.01) (xy 135.89 80.01)
+		)
+		(stroke
+			(width 0)
+			(type default)
+		)
+	)
+	(wire
+		(pts
+			(xy 119.38 72.39) (xy 135.89 72.39)
+		)
+		(stroke
+			(width 0)
+			(type default)
+		)
+	)
+	(wire
+		(pts
+			(xy 148.59 80.01) (xy 160.02 80.01)
+		)
+		(stroke
+			(width 0)
+			(type default)
+		)
+	)
+	(wire
+		(pts
+			(xy 148.59 69.85) (xy 160.02 69.85)
+		)
+		(stroke
+			(width 0)
+			(type default)
+		)
+	)
+	(wire
+		(pts
+			(xy 148.59 77.47) (xy 160.02 77.47)
 		)
 		(stroke
@@
 		(lib_id "Connector_Generic:Conn_01x05")
 		(at 165.1 80.01 0)
+		(mirror x)
 		(unit 1)
 		(body_style 1)
@@
 		(dnp no)
 		(property "Reference" "J7"
-			(at 167.64 78.7399 0)
+			(at 167.64 81.2801 0)
 			(show_name no)
 			(do_not_autoplace no)
@@
 		)
 		(property "Value" "Conn_01x05"
-			(at 167.64 81.2799 0)
+			(at 167.64 78.7401 0)
 			(show_name no)
 			(do_not_autoplace no)
@@
 		(lib_id "Connector_Generic:Conn_01x05")
 		(at 165.1 67.31 0)
+		(mirror x)
 		(unit 1)
 		(body_style 1)
@@
 		(dnp no)
 		(property "Reference" "J6"
-			(at 167.64 66.0399 0)
+			(at 167.64 68.5801 0)
 			(show_name no)
 			(do_not_autoplace no)
@@
 		)
 		(property "Value" "Conn_01x05"
-			(at 167.64 68.5799 0)
-			(show_name no)
-			(do_not_autoplace no)
+			(at 167.64 66.0401 0)
+			(show_name no)
+			(do_not_autoplace no)
